File: pcb/FS-CAN/FS-CAN.kicad_sch (KiCad schematic)
At the start: 38 parts, among them J1 USB_C_Plug_USB2.0, J2 Conn_01x02, U1 NCP1117-3.3_SOT223, U2 W25Q128JVS, U3 RP2040, U4 MCP2517FD-xSL, U5 MCP2562-E-SN, Y1 ABLS-12.000MHZ-B4-T

Commit message: 2nd CAN bus
2nd CAN bus, connector idea (only semi related)
Parts:
- added C21, C22, C23, C24: 22p, Capacitor_SMD:C_0402_1005Metric, symbol Device:C
- added C25, C26: 100n, Capacitor_SMD:C_0402_1005Metric, symbol Device:C
- added C27, C28: 4.7u, Capacitor_SMD:C_0402_1005Metric, symbol Device:C
- added J3, J4: Screw_Terminal_01x03, symbol Connector:Screw_Terminal_01x03
- added JP1, JP2: Terminating, symbol Jumper:Jumper_2_Open
- added R7: 120, Capacitor_SMD:C_0402_1005Metric, symbol Device:R
- added U6: MCP2517FD-xSL, Package_SO:SOIC-14_3.9x8.7mm_P1.27mm, symbol Interface_CAN_LIN:MCP2517FD-xSL
- added U7: MCP2562-E-SN, Package_SO:SOIC-8_3.9x4.9mm_P1.27mm, symbol Interface_CAN_LIN:MCP2562-E-SN
- added Y2, Y3: 40MHz Crystal, symbol Device:Crystal_GND24_Small
- R6: value 6k8 -> 120
Connections:
- net +3V3: now also C25.1, C26.1, U6.14 (VDD), U7.5 (Vio); no longer R6.1
- net GND: now also C21.2, C22.2, C23.2, C24.2, C25.2, C26.2, C27.2, C28.2, J3.2 (Pin_2), J4.2 (Pin_2), U6.7 (VSS), U7.2 (VSS), Y2.2, Y2.4, Y3.2, Y3.4
- net IRQ: now also U6.4 (~{INT})
- net SOF: now also U6.3 (CLKO/SOF)
- net SPI1_Rx: now also U6.12 (SDO)
- net SPI1_SCK: now also U6.10 (SCK)
- net SPI1_Tx: now also U6.11 (SDI)
- net VBUS: now also C27.1, C28.1, U7.3 (VDD)
- net at U4.1 (TXCAN), U5.1 (TXD): no longer R6.2
- net at U5.6 (CANL): now also J3.3 (Pin_3), R7.2
- net at U5.7 (CANH): now also J3.1 (Pin_1), JP1.2 (B)
- net at U4.5 (OSC2): now also C21.1, Y2.1
- net at U4.6 (OSC1): now also C22.1, Y2.3
- net CSn renamed CSn1
- net GPIO7 renamed CSn2
- net CSn2: now also U6.13 (nCS)
- new net: JP1.1 (A), R7.1
- new net: U6.1 (TXCAN), U7.1 (TXD)
- new net: U6.2 (RXCAN), U7.4 (RXD)
- new net: J4.3 (Pin_3), R6.2, U7.6 (CANL)
- new net: J4.1 (Pin_1), JP2.2 (B), U7.7 (CANH)
- new net: C23.1, U6.5 (OSC2), Y3.1
- new net: C24.1, U6.6 (OSC1), Y3.3
- new net: JP2.1 (A), R6.1
Other:
- note added: "https://www.digikey.com/en/products/detail/jst-sales-america-inc/A08SR08SR30K51A/6009376 https://www.digikey.com/en/products/detail/jst-sales-america-inc/SM08B-SRSS-TB-LF-SN/926714"
- moved on the sheet: C17, C18, C19, C20, U4, U5
